File: Nixie clock/Nixie clock.brd (EAGLE design)
At the start: 184.1 x 108.9 mm, 112 parts, among them IC1 74141N, IC10 74HC595D, IC11 SN74ALVC164245DGGR, IC12 LM555D, IC13 DS3231/SO, IC2 74141N, IC3 74141N, IC4 74141N, IC5 74141N, IC6 74141N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

Commit message: Included SHT20 code
Routing:
- net N$80: track 48.6 -> 42.7 mm
- net N$27: track 31.9 -> 26.7 mm
Changed lines of the file:
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@@
 <contactref element="N2" pad="7"/>
 <contactref element="IC2" pad="10"/>
-<wire x1="65.7453" y1="75.3768" x2="67.8385" y2="77.47" width="0.3048" layer="16"/>
-<wire x1="73.66" y1="77.47" x2="77.47" y2="73.66" width="0.3048" layer="16"/>
-<wire x1="67.8385" y1="77.47" x2="73.66" y2="77.47" width="0.3048" layer="16"/>
-<wire x1="77.47" y1="73.66" x2="77.47" y2="55.88" width="0.3048" layer="16"/>
+<wire x1="69.85" y1="66.9925" x2="69.85" y2="75.2475" width="0.3048" layer="16"/>
+<wire x1="69.85" y1="75.2475" x2="69.7207" y2="75.3768" width="0.3048" layer="16"/>
+<wire x1="69.7207" y1="75.3768" x2="65.7453" y2="75.3768" width="0.3048" layer="16"/>
+<wire x1="77.47" y1="55.88" x2="77.47" y2="59.3725" width="0.3048" layer="16"/>
+<wire x1="77.47" y1="59.3725" x2="69.85" y2="66.9925" width="0.3048" layer="16"/>
 </signal>
 <signal name="N$28">
 <contactref element="IC2" pad="11"/>
 <contactref element="N2" pad="6"/>
-<wire x1="68.3687" y1="62.23" x2="68.3687" y2="73.9999" width="0.3048" layer="16"/>
-<wire x1="74.93" y1="55.88" x2="74.7187" y2="55.88" width="0.3048" layer="16"/>
-<wire x1="74.7187" y1="55.88" x2="68.3687" y2="62.23" width="0.3048" layer="16"/>
+<wire x1="68.3687" y1="66.04" x2="68.3687" y2="73.9999" width="0.3048" layer="16"/>
+<wire x1="74.93" y1="55.88" x2="74.93" y2="59.4787" width="0.3048" layer="16"/>
+<wire x1="74.93" y1="59.4787" x2="68.3687" y2="66.04" width="0.3048" layer="16"/>
 </signal>
 <signal name="N$29">
@@
 <contactref element="IC8" pad="8"/>
 <contactref element="N11" pad="10"/>
-<wire x1="198.12" y1="72.39" x2="208.28" y2="72.39" width="0.3048" layer="16"/>
 <wire x1="191.076" y1="82.7479" x2="194.857240625" y2="78.966659375" width="0.3048" layer="16"/>
-<wire x1="208.28" y1="72.39" x2="209.55" y2="71.12" width="0.3048" layer="16"/>
-<wire x1="209.55" y1="71.12" x2="209.55" y2="50.8" width="0.3048" layer="16"/>
+<wire x1="209.55" y1="58.7375" x2="209.55" y2="50.8" width="0.3048" layer="16"/>
 <wire x1="209.55" y1="50.8" x2="208.28" y2="49.53" width="0.3048" layer="16"/>
 <wire x1="208.28" y1="49.53" x2="208.28" y2="48.26" width="0.3048" layer="16"/>
-<wire x1="194.857240625" y1="75.652759375" x2="194.857240625" y2="78.966659375" width="0.3048" layer="16"/>
-<wire x1="198.12" y1="72.39" x2="194.857240625" y2="75.652759375" width="0.3048" layer="16"/>
+<wire x1="194.857240625" y1="78.966659375" x2="194.857240625" y2="73.430259375" width="0.3048" layer="16"/>
+<wire x1="194.857240625" y1="73.430259375" x2="209.55" y2="58.7375" width="0.3048" layer="16"/>
 </signal>
 <signal name="N$81">
